Commit message: Configure the Differential Drive Controller with ROS2 Control

File: cp15_auxiliary_files/rb1_ros2_description/xacro/rb1_ros2_base.urdf.xacro (robot description, xacro)
@@ -84,5 +84,33 @@
 		<origin xyz="0.234 0.0 0.092" rpy="0 0 0"/>
 	</xacro:sensor_orbbec_astra>
-	<!-- Gazebo ros2 control plugins -->
 	<!-- <xacro:ros2_control/> -->
+    <ros2_control name="diff_drive" type="system">
+      <hardware>
+          <plugin>gazebo_ros2_control/GazeboSystem</plugin>
+      </hardware>
+      <joint name="robot_left_wheel_joint">
+        <command_interface name="velocity">
+          <param name="min">-1</param>
+          <param name="max">1</param>
+        </command_interface>
+        <state_interface name="position"/>
+        <state_interface name="velocity"/>
+        <state_interface name="effort"/>
+      </joint>
+      <joint name="robot_right_wheel_joint">
+        <command_interface name="velocity">
+          <param name="min">-1</param>
+          <param name="max">1</param>
+        </command_interface>
+        <state_interface name="position"/>
+        <state_interface name="velocity"/>
+        <state_interface name="effort"/>
+      </joint>
+    </ros2_control>
+    <!-- Gazebo ros2 control plugins -->
+    <gazebo>
+        <plugin filename="libgazebo_ros2_control.so" name="gazebo_ros2_control">
+        <parameters>$(find rb1_ros2_description)/config/rb1_controller.yaml</parameters>
+        </plugin>
+  </gazebo>
 </robot>

Commit message: Implement a ROS2 Controller to have a functional Lifting Unit

File: cp15_auxiliary_files/rb1_ros2_description/xacro/rb1_ros2_base.urdf.xacro (robot description, xacro)
@@ -111,6 +111,25 @@
     <gazebo>
         <plugin filename="libgazebo_ros2_control.so" name="gazebo_ros2_control">
+            <parameters>$(find rb1_ros2_description)/config/rb1_controller.yaml</parameters>
+        </plugin>
+    </gazebo>
+    <ros2_control name="effort_controllers" type="system">
+        <hardware>
+            <plugin>gazebo_ros2_control/GazeboSystem</plugin>
+        </hardware>
+        <joint name="robot_elevator_platform_joint">
+            <command_interface name="effort">
+                <param name="min">-10</param>
+                <param name="max">10</param>
+            </command_interface>
+            <state_interface name="position"/>
+            <state_interface name="velocity"/>
+            <state_interface name="effort"/>
+        </joint>
+  </ros2_control>
+  <gazebo>
+    <plugin filename="libgazebo_ros_force_system.so" name="gazebo_ros2_control">
         <parameters>$(find rb1_ros2_description)/config/rb1_controller.yaml</parameters>
-        </plugin>
+    </plugin>
   </gazebo>
 </robot>
